Commit message: Part1 Fixed

File: adventure_simulator/adventure_description/urdf/sensors/asus_xtion_pro.urdf.xacro (robot description, xacro)
@@ -7,7 +7,8 @@
   <xacro:property name="asus_xtion_pro_depth_rel_rgb_py" value="0.0270" />
   <xacro:property name="asus_xtion_pro_cam_rel_rgb_py"   value="-0.0220" />
-  <xacro:macro name="sensor_asus_xtion_pro" params="parent">
+  <xacro:macro name="sensor_asus_xtion_pro" params="parent *origin">
     <joint name="camera_rgb_joint" type="fixed">
-        <origin xyz="0 0 0.3" rpy="0 0 0"/>
+        <!--<origin xyz="0 0 0.1" rpy="0 0 0"/>-->
+      <xacro:insert_block name="origin" />
       <parent link="${parent}"/>
       <child link="camera_rgb_frame" />
